Commit message: update spm

File: config/spm_3dof.urdf_old.xacro (robot description, xacro)
@@ -3,20 +3,14 @@
     <!-- This will include all the contents of example_include.xacro first. Go check it out! -->
     <xacro:include filename="example_include.xacro" />
-    <!-- Load spm_3dof geometric parameters: -->
-    <xacro:arg name="r_c" default="1.0" />
-    <xacro:arg name="ang_b_m" default="1.0" />
+    <!-- Load spherical robot geometric parameters: -->
     <xacro:arg name="r_b" default="1.0" />
-    <xacro:arg name="r_s_out" default="1.0" />
-    <xacro:arg name="d" default="1.0" />
-    <xacro:arg name="r_e" default="1.0" />
-    <xacro:arg name="r_s_in" default="1.0" />
+    <xacro:arg name="ratio_c_b" default="1.0" />
+    <xacro:arg name="ratio_e_b" default="1.0" />
     <!-- Convert them into xacro properties: -->
-    <xacro:property name="r_c" value="$(arg r_c)" />
-    <xacro:property name="ang_b_m" value="$(arg ang_b_m)" />
     <xacro:property name="r_b" value="$(arg r_b)" />
-    <xacro:property name="r_s_out" value="$(arg r_s_out)" />
-    <xacro:property name="d" value="$(arg d)" />
-    <xacro:property name="r_e" value="$(arg r_e)" />
-    <xacro:property name="r_s_in" value="$(arg r_s_in)" />
+    <xacro:property name="ratio_c_b" value="$(arg ratio_c_b)" />
+    <xacro:property name="ratio_e_b" value="$(arg ratio_e_b)" />
+    <xacro:property name="r_c" value="$(eval ratio_c_b * r_b)"/>
+    <xacro:property name="r_e" value="$(eval ratio_e_b * r_b)"/>
     <!-- world -->
     <link name="world"></link>
@@ -54,7 +48,7 @@
             <geometry>
                 <mesh filename="package://cga_ik/meshes/arc_link_thin.stl"
-                    scale="${r_s_in}
-                           ${r_s_in}
-                           ${r_s_in}"/>
+                    scale="${ sqrt(r_b * r_b  + r_c * r_c) }
+                           ${ sqrt(r_b * r_b  + r_c * r_c) }
+                           ${ sqrt(r_b * r_b  + r_c * r_c) }"/>
             </geometry>
             <material name="white" />
@@ -73,7 +67,7 @@
             <geometry>
                 <mesh filename="package://cga_ik/meshes/arc_link_thin.stl"
-                    scale="${r_s_in}
-                           ${r_s_in}
-                           ${r_s_in}"/>
+                    scale="${ sqrt(r_b * r_b  + r_c * r_c) }
+                           ${ sqrt(r_b * r_b  + r_c * r_c) }
+                           ${ sqrt(r_b * r_b  + r_c * r_c) }"/>
             </geometry>
             <material name="white" />
@@ -92,7 +86,7 @@
             <geometry>
                 <mesh filename="package://cga_ik/meshes/arc_link_thin.stl"
-                    scale="${r_s_in}
-                           ${r_s_in}
-                           ${r_s_in}"/>
+                    scale="${ sqrt(r_b * r_b  + r_c * r_c) }
+                           ${ sqrt(r_b * r_b  + r_c * r_c) }
+                           ${ sqrt(r_b * r_b  + r_c * r_c) }"/>
             </geometry>
             <material name="white" />
@@ -111,7 +105,7 @@
             <geometry>
                 <mesh filename="package://cga_ik/meshes/arc_link_thin.stl"
-                    scale="${r_s_in}
-                           ${r_s_in}
-                           ${r_s_in}"/>
+                    scale="${ sqrt(r_b * r_b  + r_c * r_c) }
+                           ${ sqrt(r_b * r_b  + r_c * r_c) }
+                           ${ sqrt(r_b * r_b  + r_c * r_c) }"/>
             </geometry>
             <material name="white" />
@@ -130,7 +124,7 @@
             <geometry>
                 <mesh filename="package://cga_ik/meshes/arc_link_thin.stl"
-                    scale="${r_s_in}
-                           ${r_s_in}
-                           ${r_s_in}"/>
+                    scale="${ sqrt(r_b * r_b  + r_c * r_c) }
+                           ${ sqrt(r_b * r_b  + r_c * r_c) }
+                           ${ sqrt(r_b * r_b  + r_c * r_c) }"/>
             </geometry>
             <material name="white" />
@@ -149,7 +143,7 @@
             <geometry>
                 <mesh filename="package://cga_ik/meshes/arc_link_thin.stl"
-                    scale="${r_s_in}
-                           ${r_s_in}
-                           ${r_s_in}"/>
+                    scale="${ sqrt(r_b * r_b  + r_c * r_c) }
+                           ${ sqrt(r_b * r_b  + r_c * r_c) }
+                           ${ sqrt(r_b * r_b  + r_c * r_c) }"/>
             </geometry>
             <material name="white" />
