Commit message: update spm urdf and meshes; add krl for left or right elbow configs

File: config/spm_3dof_simplified.urdf.xacro (robot description, xacro)
@@ -31,6 +31,6 @@
             <origin xyz="0 0 0" rpy="0 0 0"/>
             <geometry>
-                <mesh filename="package://cga_ik/meshes/spm_3dof/spm_base_plate.stl"
-                      scale="${mm2m} ${mm2m} ${mm2m}"/>
+                <mesh filename="package://cga_ik/meshes/spm_3dof/base_plate.stl"
+                      scale="${r_b} ${r_b} ${r_b}"/>
             </geometry>
             <material name="white" />
@@ -56,6 +56,8 @@
             <origin xyz="0 0 0" rpy="0 0 ${pi}"/>
             <geometry>
-                <mesh filename="package://cga_ik/meshes/spm_3dof/spm_motor_link.stl"
-                    scale="${mm2m} ${mm2m} ${mm2m}"/>
+                <mesh filename="package://cga_ik/meshes/spm_3dof/arc_link_thin.stl"
+                    scale="${r_s_m}
+                           ${r_s_m}
+                           ${r_s_m}"/>
             </geometry>
             <material name="white" />
@@ -73,6 +75,8 @@
             <origin xyz="0 0 0" rpy="0 0 ${pi}"/>
             <geometry>
-                <mesh filename="package://cga_ik/meshes/spm_3dof/spm_motor_link.stl"
-                    scale="${mm2m} ${mm2m} ${mm2m}"/>
+                <mesh filename="package://cga_ik/meshes/spm_3dof/arc_link_thin.stl"
+                    scale="${r_s_m}
+                           ${r_s_m}
+                           ${r_s_m}"/>
             </geometry>
             <material name="white" />
@@ -90,6 +94,8 @@
             <origin xyz="0 0 0" rpy="0 0 ${pi}"/>
             <geometry>
-                <mesh filename="package://cga_ik/meshes/spm_3dof/spm_motor_link.stl"
-                    scale="${mm2m} ${mm2m} ${mm2m}"/>
+                <mesh filename="package://cga_ik/meshes/spm_3dof/arc_link_thin.stl"
+                    scale="${r_s_m}
+                           ${r_s_m}
+                           ${r_s_m}"/>
             </geometry>
             <material name="white" />
@@ -105,8 +111,10 @@
     <link name="spm_elbow_0">
         <visual>
-            <origin xyz="0 0 0" rpy="${pi} 0 0"/>
+            <origin xyz="0 0 0" rpy="0 0 0"/>
             <geometry>
-                <mesh filename="package://cga_ik/meshes/spm_3dof/spm_elbow_link.stl"
-                    scale="${mm2m} ${mm2m} ${mm2m}"/>
+                <mesh filename="package://cga_ik/meshes/spm_3dof/arc_link_thin.stl"
+                    scale="${r_s_elb}
+                           ${r_s_elb}
+                           ${r_s_elb}"/>
             </geometry>
             <material name="white" />
@@ -122,8 +130,10 @@
     <link name="spm_elbow_1">
         <visual>
-            <origin xyz="0 0 0" rpy="${pi} 0 0"/>
+            <origin xyz="0 0 0" rpy="0 0 0"/>
             <geometry>
-                <mesh filename="package://cga_ik/meshes/spm_3dof/spm_elbow_link.stl"
-                    scale="${mm2m} ${mm2m} ${mm2m}"/>
+                <mesh filename="package://cga_ik/meshes/spm_3dof/arc_link_thin.stl"
+                    scale="${r_s_elb}
+                           ${r_s_elb}
+                           ${r_s_elb}"/>
             </geometry>
             <material name="white" />
@@ -139,8 +149,10 @@
     <link name="spm_elbow_2">
         <visual>
-            <origin xyz="0 0 0" rpy="${pi} 0 0"/>
+            <origin xyz="0 0 0" rpy="0 0 0"/>
             <geometry>
-                <mesh filename="package://cga_ik/meshes/spm_3dof/spm_elbow_link.stl"
-                    scale="${mm2m} ${mm2m} ${mm2m}"/>
+                <mesh filename="package://cga_ik/meshes/spm_3dof/arc_link_thin.stl"
+                    scale="${r_s_elb}
+                           ${r_s_elb}
+                           ${r_s_elb}"/>
             </geometry>
             <material name="white" />
@@ -158,6 +170,6 @@
             <origin xyz="0 0 0" rpy="0 0 0"/>
             <geometry>
-                <mesh filename="package://cga_ik/meshes/spm_3dof/spm_end_plate.stl"
-                      scale="${mm2m} ${mm2m} ${mm2m}"/>
+                <mesh filename="package://cga_ik/meshes/spm_3dof/end_plate.stl"
+                      scale="${r_e} ${r_e} ${r_e}"/>
             </geometry>
             <material name="white" />
