Commit message: update spm_3dof

File: config/spm_3dof.urdf.xacro (robot description, xacro)
@@ -1,4 +1,4 @@
 <?xml version="1.0"?>
-<robot xmlns:xacro="http://www.ros.org/wiki/xacro"  name="robot">
+<robot xmlns:xacro="http://www.ros.org/wiki/xacro"  name="spm_3dof">
     <!-- This will include all the contents of example_include.xacro first. Go check it out! -->
     <xacro:include filename="example_include.xacro" />
@@ -16,5 +16,5 @@
     <link name="world"></link>
     <!-- base -->
-    <link name="srb_base">
+    <link name="spm_base">
         <visual>
             <origin xyz="0 0 0" rpy="0 0 0"/>
@@ -31,17 +31,17 @@
     <joint name="joint_world_base" type="fixed">
         <parent link="world"/>
-        <child link="srb_base"/>
+        <child link="spm_base"/>
         <origin xyz="0 0 0" rpy="0 0 0"/>
     </joint>
     <!-- rot_cen -->
-    <link name="srb_rot_cen"></link>
+    <link name="spm_rot_cen"></link>
     <!-- base to rot_cen -->
     <joint name="joint_base_rot_cen" type="floating">
-        <parent link="srb_base"/>
-        <child link="srb_rot_cen"/>
+        <parent link="spm_base"/>
+        <child link="spm_rot_cen"/>
         <origin xyz="0 0 0" rpy="0 0 0"/>
     </joint>
     <!-- motor_0 -->
-    <link name="srb_motor_0">
+    <link name="spm_motor_0">
         <visual>
             <origin xyz="0 0 0" rpy="0 0 0"/>
@@ -57,10 +57,10 @@
     <!-- rot_cen to motor_0 -->
     <joint name="joint_rot_cen_motor_0" type="floating">
-        <parent link="srb_rot_cen"/>
-        <child link="srb_motor_0"/>
+        <parent link="spm_rot_cen"/>
+        <child link="spm_motor_0"/>
         <origin xyz="0 0 0" rpy="0 0 0"/>
     </joint>
     <!-- motor_1 -->
-    <link name="srb_motor_1">
+    <link name="spm_motor_1">
         <visual>
             <origin xyz="0 0 0" rpy="0 0 0"/>
@@ -76,10 +76,10 @@
     <!-- rot_cen to motor_1 -->
     <joint name="joint_rot_cen_motor_1" type="floating">
-        <parent link="srb_rot_cen"/>
-        <child link="srb_motor_1"/>
+        <parent link="spm_rot_cen"/>
+        <child link="spm_motor_1"/>
         <origin xyz="0 0 0" rpy="0 0 0"/>
     </joint>
     <!-- motor_2 -->
-    <link name="srb_motor_2">
+    <link name="spm_motor_2">
         <visual>
             <origin xyz="0 0 0" rpy="0 0 0"/>
@@ -95,10 +95,10 @@
     <!-- rot_cen to motor_2 -->
     <joint name="joint_rot_cen_motor_2" type="floating">
-        <parent link="srb_rot_cen"/>
-        <child link="srb_motor_2"/>
+        <parent link="spm_rot_cen"/>
+        <child link="spm_motor_2"/>
         <origin xyz="0 0 0" rpy="0 0 0"/>
     </joint>
     <!-- elbow_0 -->
-    <link name="srb_elbow_0">
+    <link name="spm_elbow_0">
         <visual>
             <origin xyz="0 0 0" rpy="0 0 0"/>
@@ -114,10 +114,10 @@
     <!-- rot_cen to elbow_0 -->
     <joint name="joint_rot_cen_elbow_0" type="floating">
-        <parent link="srb_rot_cen"/>
-        <child link="srb_elbow_0"/>
+        <parent link="spm_rot_cen"/>
+        <child link="spm_elbow_0"/>
         <origin xyz="0 0 0" rpy="0 0 0"/>
     </joint>
     <!-- elbow_1 -->
-    <link name="srb_elbow_1">
+    <link name="spm_elbow_1">
         <visual>
             <origin xyz="0 0 0" rpy="0 0 0"/>
@@ -133,10 +133,10 @@
     <!-- rot_cen to elbow_1 -->
     <joint name="joint_rot_cen_elbow_1" type="floating">
-        <parent link="srb_rot_cen"/>
-        <child link="srb_elbow_1"/>
+        <parent link="spm_rot_cen"/>
+        <child link="spm_elbow_1"/>
         <origin xyz="0 0 0" rpy="0 0 0"/>
     </joint>
     <!-- elbow_2 -->
-    <link name="srb_elbow_2">
+    <link name="spm_elbow_2">
         <visual>
             <origin xyz="0 0 0" rpy="0 0 0"/>
@@ -152,10 +152,10 @@
     <!-- rot_cen to elbow_2 -->
     <joint name="joint_rot_cen_elbow_2" type="floating">
-        <parent link="srb_rot_cen"/>
-        <child link="srb_elbow_2"/>
+        <parent link="spm_rot_cen"/>
+        <child link="spm_elbow_2"/>
         <origin xyz="0 0 0" rpy="0 0 0"/>
     </joint>
     <!-- epl_c -->
-    <link name="srb_epl_c">
+    <link name="spm_epl_c">
         <visual>
             <origin xyz="0 0 0" rpy="0 0 0"/>
@@ -171,6 +171,6 @@
     <!-- rot_cen to epl_c -->
     <joint name="joint_rot_cen_epl_c" type="floating">
-        <parent link="srb_rot_cen"/>
-        <child link="srb_epl_c"/>
+        <parent link="spm_rot_cen"/>
+        <child link="spm_epl_c"/>
         <origin xyz="0 0 0" rpy="0 0 0"/>
     </joint>

Commit message: update spm

File: config/spm_3dof.urdf.xacro (robot description, xacro)
@@ -11,4 +11,5 @@
     <xacro:arg name="r_e" default="1.0" />
     <xacro:arg name="r_s_in" default="1.0" />
+    <xacro:arg name="r_s_elb" default="1.0" />
     <!-- Convert them into xacro properties: -->
     <xacro:property name="r_c" value="$(arg r_c)" />
@@ -19,4 +20,5 @@
     <xacro:property name="r_e" value="$(arg r_e)" />
     <xacro:property name="r_s_in" value="$(arg r_s_in)" />
+    <xacro:property name="r_s_elb" value="$(arg r_s_elb)" />
     <!-- world -->
     <link name="world"></link>
@@ -111,7 +113,7 @@
             <geometry>
                 <mesh filename="package://cga_ik/meshes/arc_link_thin.stl"
-                    scale="${r_s_in}
-                           ${r_s_in}
-                           ${r_s_in}"/>
+                    scale="${r_s_elb}
+                           ${r_s_elb}
+                           ${r_s_elb}"/>
             </geometry>
             <material name="white" />
@@ -130,7 +132,7 @@
             <geometry>
                 <mesh filename="package://cga_ik/meshes/arc_link_thin.stl"
-                    scale="${r_s_in}
-                           ${r_s_in}
-                           ${r_s_in}"/>
+                    scale="${r_s_elb}
+                           ${r_s_elb}
+                           ${r_s_elb}"/>
             </geometry>
             <material name="white" />
@@ -149,7 +151,7 @@
             <geometry>
                 <mesh filename="package://cga_ik/meshes/arc_link_thin.stl"
-                    scale="${r_s_in}
-                           ${r_s_in}
-                           ${r_s_in}"/>
+                    scale="${r_s_elb}
+                           ${r_s_elb}
+                           ${r_s_elb}"/>
             </geometry>
             <material name="white" />

Commit message: update spm

File: config/spm_3dof.urdf.xacro (robot description, xacro)
@@ -156,5 +156,5 @@
     <link name="spm_epl_c">
         <visual>
-            <origin xyz="0 0 0" rpy="0 0 0"/>
+            <origin xyz="0 0 ${-13.24849 * mm2m}" rpy="0 0 ${-(1.0 / 6.0) * pi}"/>
             <geometry>
                 <mesh filename="package://cga_ik/meshes/spm_3dof/spm_end_plate.stl"

Commit message: update spm

File: config/spm_3dof.urdf.xacro (robot description, xacro)
@@ -13,4 +13,5 @@
     <xacro:arg name="r_s_elb" default="1.0" />
     <xacro:arg name="r_s_epl" default="1.0" />
+    <xacro:arg name="th_z_ee_init" default="1.0" />
     <!-- Convert them into xacro properties: -->
     <xacro:property name="mm2m" value="0.001" />
@@ -24,4 +25,5 @@
     <xacro:property name="r_s_elb" value="$(arg r_s_elb)" />
     <xacro:property name="r_s_epl" value="$(arg r_s_epl)" />
+    <xacro:property name="th_z_ee_init" value="$(arg th_z_ee_init)" />
     <!-- world -->
     <link name="world"></link>

Commit message: update spm

File: config/spm_3dof.urdf.xacro (robot description, xacro)
@@ -13,5 +13,5 @@
     <xacro:arg name="r_s_elb" default="1.0" />
     <xacro:arg name="r_s_epl" default="1.0" />
-    <xacro:arg name="th_z_ee_init" default="1.0" />
+    <xacro:arg name="th_z_ee_reset" default="1.0" />
     <!-- Convert them into xacro properties: -->
     <xacro:property name="mm2m" value="0.001" />
@@ -25,5 +25,5 @@
     <xacro:property name="r_s_elb" value="$(arg r_s_elb)" />
     <xacro:property name="r_s_epl" value="$(arg r_s_epl)" />
-    <xacro:property name="th_z_ee_init" value="$(arg th_z_ee_init)" />
+    <xacro:property name="th_z_ee_reset" value="$(arg th_z_ee_reset)" />
     <!-- world -->
     <link name="world"></link>

Commit message: update spm

File: config/spm_3dof.urdf.xacro (robot description, xacro)
@@ -33,5 +33,5 @@
             <origin xyz="0 0 0" rpy="0 0 0"/>
             <geometry>
-                <mesh filename="package://cga_ik/meshes/spm_3dof/spm_base_plate.stl"
+                <mesh filename="package://cga_ik/meshes/spm_3dof/spm_base_plate_with_blocks_and_motors.stl"
                       scale="${mm2m} ${mm2m} ${mm2m}"/>
             </geometry>
@@ -58,5 +58,5 @@
             <origin xyz="0 0 0" rpy="0 0 ${pi}"/>
             <geometry>
-                <mesh filename="package://cga_ik/meshes/spm_3dof/spm_motor_link.stl"
+                <mesh filename="package://cga_ik/meshes/spm_3dof/spm_motor_link_with_pulley.stl"
                     scale="${mm2m} ${mm2m} ${mm2m}"/>
             </geometry>
@@ -75,5 +75,5 @@
             <origin xyz="0 0 0" rpy="0 0 ${pi}"/>
             <geometry>
-                <mesh filename="package://cga_ik/meshes/spm_3dof/spm_motor_link.stl"
+                <mesh filename="package://cga_ik/meshes/spm_3dof/spm_motor_link_with_pulley.stl"
                     scale="${mm2m} ${mm2m} ${mm2m}"/>
             </geometry>
@@ -92,5 +92,5 @@
             <origin xyz="0 0 0" rpy="0 0 ${pi}"/>
             <geometry>
-                <mesh filename="package://cga_ik/meshes/spm_3dof/spm_motor_link.stl"
+                <mesh filename="package://cga_ik/meshes/spm_3dof/spm_motor_link_with_pulley.stl"
                     scale="${mm2m} ${mm2m} ${mm2m}"/>
             </geometry>
