Commit message: update namings

File: config/tm5-700.urdf.xacro (robot description, xacro)
@@ -34,5 +34,5 @@
     <!-- If Arm is fixed to world -->
     <joint name="base_joint" type="fixed">
-      <origin xyz="0 0 0" rpy="0 0 0" />
+      <origin xyz="0 -0.5 0" rpy="0 0 0" />
       <parent link="world" />
       <child link="base" />

Commit message: update readme

File: config/tm5-700.urdf.xacro (robot description, xacro)
@@ -34,5 +34,5 @@
     <!-- If Arm is fixed to world -->
     <joint name="base_joint" type="fixed">
-      <origin xyz="0 -0.5 0" rpy="0 0 0" />
+      <origin xyz="0 0 0" rpy="0 0 0" />
       <parent link="world" />
       <child link="base" />
