Commit message: update xacro files and readme

File: config/intertias.xacro (robot description, xacro)
@@ -1,20 +1,5 @@
 <?xml version="1.0"?>
 <robot xmlns:xacro="http://www.ros.org/wiki/xacro" >
-    <!-- This file is not a robot in and of itself, it just contains some useful tags that could be included in any robot -->
-    <!-- Specify some colours -->
-    <material name="white">
-        <color rgba="1 1 1 1"/>
-    </material>
-    <material name="orange">
-        <color rgba="1 0.3 0.1 1"/>
-    </material>
-    <material name="blue">
-        <color rgba="0.2 0.2 1 1"/>
-    </material>
-    <material name="green">
-        <color rgba="0.2 1 0.2 1"/>
-    </material>
-    <!-- Specify some standard inertial calculations https://en.wikipedia.org/wiki/List_of_moments_of_inertia -->
-    <!-- These make use of xacro's mathematical functionality -->
+    <!-- See details at: https://en.wikipedia.org/wiki/List_of_moments_of_inertia -->
     <xacro:macro name="inertial_sphere" params="mass radius *origin">
         <inertial>

File: config/spm_3dof.urdf.xacro (robot description, xacro)
@@ -1,6 +1,6 @@
 <?xml version="1.0"?>
 <robot xmlns:xacro="http://www.ros.org/wiki/xacro"  name="spm_3dof">
-    <!-- This will include all the contents of example_include.xacro first. Go check it out! -->
-    <xacro:include filename="example_include.xacro" />
+    <!-- Load properties defined in other xacro files -->
+    <xacro:include filename="colors.xacro" />
     <!-- Load spm_3dof geometric parameters: -->
     <xacro:arg name="r_c" default="1.0" />

File: config/tm5-700.srdf.xacro (robot description, xacro)
@@ -66,36 +66,3 @@
     <disable_collisions link1="link_4" link2="link_6" reason="Never"/>
     <disable_collisions link1="link_5" link2="link_6" reason="Adjacent"/>
-    <!-- <disable_collisions link1="link_6" link2="robotiq_85_base_link" reason="Adjacent"/> -->
-    <!-- <disable_collisions link1="link_6" link2="tm5-700rs_adapter" reason="Adjacent"/>
-    <disable_collisions link1="tm5-700rs_adapter" link2="camera_bottom_screw_frame" reason="Adjacent"/>
-    <disable_collisions link1="camera_bottom_screw_frame" link2="camera_link" reason="Never"/>
-    <disable_collisions link1="tm5-700rs_adapter" link2="robotiq_85_base_link" reason="Adjacent"/> -->
-    <!-- <disable_collisions link1="robotiq_85_base_link" link2="robotiq_85_left_knuckle_link" reason="Adjacent"/>
-    <disable_collisions link1="robotiq_85_base_link" link2="robotiq_85_right_knuckle_link" reason="Adjacent"/>
-    <disable_collisions link1="robotiq_85_base_link" link2="robotiq_85_left_finger_link" reason="Never"/>
-    <disable_collisions link1="robotiq_85_base_link" link2="robotiq_85_right_finger_link" reason="Never"/>
-    <disable_collisions link1="robotiq_85_base_link" link2="robotiq_85_left_inner_knuckle_link" reason="Never"/>
-    <disable_collisions link1="robotiq_85_base_link" link2="robotiq_85_right_inner_knuckle_link" reason="Never"/>
-    <disable_collisions link1="robotiq_85_base_link" link2="robotiq_85_left_finger_tip_link" reason="Never"/>
-    <disable_collisions link1="robotiq_85_base_link" link2="robotiq_85_right_finger_tip_link" reason="Never"/>
-    <disable_collisions link1="robotiq_85_left_knuckle_link" link2="robotiq_85_left_finger_link" reason="Adjacent"/>
-    <disable_collisions link1="robotiq_85_right_knuckle_link" link2="robotiq_85_right_finger_link" reason="Adjacent"/>
-    <disable_collisions link1="robotiq_85_right_finger_link" link2="robotiq_85_left_finger_link" reason="Never"/>
-    <disable_collisions link1="robotiq_85_right_knuckle_link" link2="robotiq_85_left_knuckle_link" reason="Never"/>
-    <disable_collisions link1="robotiq_85_right_finger_link" link2="robotiq_85_left_knuckle_link" reason="Never"/>
-    <disable_collisions link1="robotiq_85_left_finger_link" link2="robotiq_85_right_knuckle_link" reason="Never"/>
-    <disable_collisions link1="robotiq_85_left_finger_link" link2="robotiq_85_left_finger_tip_link" reason="Adjacent"/>
-    <disable_collisions link1="robotiq_85_right_finger_link" link2="robotiq_85_right_finger_tip_link" reason="Adjacent"/>
-    <disable_collisions link1="robotiq_85_right_inner_knuckle_link" link2="robotiq_85_right_finger_tip_link" reason="Adjacent"/>
-    <disable_collisions link1="robotiq_85_left_inner_knuckle_link" link2="robotiq_85_left_finger_tip_link" reason="Adjacent"/>
-    <disable_collisions link1="link_6" link2="robotiq_85_base_link" reason="Never"/>
-    <disable_collisions link1="link_6" link2="robotiq_85_left_knuckle_link" reason="Never"/>
-    <disable_collisions link1="link_6" link2="robotiq_85_right_knuckle_link" reason="Never"/>
-    <disable_collisions link1="link_6" link2="robotiq_85_left_finger_link" reason="Never"/>
-    <disable_collisions link1="link_6" link2="robotiq_85_right_finger_link" reason="Never"/>
-    <disable_collisions link1="link_6" link2="robotiq_85_left_finger_tip_link" reason="Never"/>
-    <disable_collisions link1="link_6" link2="robotiq_85_right_finger_tip_link" reason="Never"/>
-    <disable_collisions link1="link_6" link2="robotiq_85_left_inner_knuckle_link" reason="Never"/>
-    <disable_collisions link1="link_6" link2="robotiq_85_right_inner_knuckle_link" reason="Never"/>
-    <disable_collisions link1="robotiq_85_right_finger_tip_link" link2="robotiq_85_left_finger_tip_link" reason="Never"/> -->
 </robot>
